File: kicad/BandSelector/BandSelector.kicad_pcb (KiCad board)
At the start: 2 copper layers, 105.5 x 77.6 mm, 63 parts, among them J1 DE15_Plug_HighDensity_Mountin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, J2 POWER, J3 75915416LF, Q1 2N7000, Q2 2N7000, U1 PicoW, U2 L7805

Commit message: schematic update, get 3d images
Other:
- board text added: "V 0.0.6 2024-10-26"
- board text removed: "V 0.0.5 2024-09-26"
Changed lines of the file:
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@@
 	(title_block
 		(title "n1kdo_band_selector")
-		(date "2024-09-26")
-		(rev "0.0.5")
+		(date "2024-10-26")
+		(rev "0.0.6")
 	)
 	(layers
@@
 	(net 52 "Net-(U1-GPIO1)")
 	(net 53 "Net-(U1-GPIO14)")
-	(net 54 "unconnected-(U1-VBUS-Pad40)")
-	(net 55 "unconnected-(U1-3V3_EN-Pad37)")
-	(net 56 "unconnected-(U1-3V3_EN-Pad37)_1")
-	(net 57 "unconnected-(U1-RUN-Pad30)")
-	(net 58 "unconnected-(U1-RUN-Pad30)_1")
-	(net 59 "unconnected-(U1-ADC_VREF-Pad35)")
-	(net 60 "unconnected-(U1-ADC_VREF-Pad35)_1")
-	(net 61 "unconnected-(U1-VBUS-Pad40)_1")
-	(net 62 "unconnected-(J2-PadSHUNT)")
-	(net 63 "/DIGOUT1")
-	(net 64 "unconnected-(U1-SWDIO-Pad43)")
-	(net 65 "unconnected-(U1-SWCLK-Pad41)")
-	(net 66 "unconnected-(U1-GND-Pad42)")
-	(net 67 "/LIGHT")
-	(net 68 "Net-(D10-K)")
-	(net 69 "Net-(U1-GPIO15)")
+	(net 54 "unconnected-(U1-3V3_EN-Pad37)_1")
+	(net 55 "unconnected-(U1-RUN-Pad30)_1")
+	(net 56 "unconnected-(U1-ADC_VREF-Pad35)")
+	(net 57 "unconnected-(U1-VBUS-Pad40)_1")
+	(net 58 "unconnected-(J2-PadSHUNT)")
+	(net 59 "/DIGOUT1")
+	(net 60 "unconnected-(U1-SWDIO-Pad43)")
+	(net 61 "unconnected-(U1-SWCLK-Pad41)")
+	(net 62 "unconnected-(U1-GND-Pad42)")
+	(net 63 "/LIGHT")
+	(net 64 "Net-(D10-K)")
+	(net 65 "Net-(U1-GPIO15)")
 	(footprint "Capacitor_THT:CP_Radial_D8.0mm_P3.50mm"
 		(layer "F.Cu")
@@
 			(layer "F.Fab")
 		)
-		(fp_text user "SWDIO"
-			(at 5.5 8 90)
+		(fp_text user "SWCLK"
+			(at -1 7.5 90)
 			(layer "F.SilkS")
 			(effects
@@
 			)
 		)
-		(fp_text user "SWCLK"
-			(at -1 7.5 90)
+		(fp_text user "SWDIO"
+			(at 5.5 8 90)
 			(layer "F.SilkS")
 			(effects
@@
 			(layers "*.Cu" "*.Mask")
 			(remove_unused_layers no)
-			(net 67 "/LIGHT")
+			(net 63 "/LIGHT")
 			(pinfunction "GPIO9")
 			(pintype "bidirectional")
@@
 			)
 			(layers "F.Cu" "F.Mask")
-			(net 67 "/LIGHT")
+			(net 63 "/LIGHT")
 			(pinfunction "GPIO9")
 			(pintype "bidirectional")
@@
 			(layers "*.Cu" "*.Mask")
 			(remove_unused_layers no)
-			(net 69 "Net-(U1-GPIO15)")
+			(net 65 "Net-(U1-GPIO15)")
 			(pinfunction "GPIO15")
 			(pintype "bidirectional")
@@
 			)
 			(layers "F.Cu" "F.Mask")
-			(net 69 "Net-(U1-GPIO15)")
+			(net 65 "Net-(U1-GPIO15)")
 			(pinfunction "GPIO15")
 			(pintype "bidirectional")
@@
 			(layers "*.Cu" "*.Mask")
 			(remove_unused_layers no)
-			(net 58 "unconnected-(U1-RUN-Pad30)_1")
+			(net 55 "unconnected-(U1-RUN-Pad30)_1")
 			(pinfunction "RUN")
 			(pintype "input+no_connect")
@@
 			)
 			(layers "F.Cu" "F.Mask")
-			(net 57 "unconnected-(U1-RUN-Pad30)")
+			(net 55 "unconnected-(U1-RUN-Pad30)_1")
 			(pinfunction "RUN")
 			(pintype "input+no_connect")
@@
 			(layers "*.Cu" "*.Mask")
 			(remove_unused_layers no)
-			(net 59 "unconnected-(U1-ADC_VREF-Pad35)")
+			(net 56 "unconnected-(U1-ADC_VREF-Pad35)")
 			(pinfunction "ADC_VREF")
 			(pintype "bidirectional+no_connect")
@@
 			)
 			(layers "F.Cu" "F.Mask")
-			(net 60 "unconnected-(U1-ADC_VREF-Pad35)_1")
+			(net 56 "unconnected-(U1-ADC_VREF-Pad35)")
 			(pinfunction "ADC_VREF")
 			(pintype "bidirectional+no_connect")
@@
 			(layers "*.Cu" "*.Mask")
 			(remove_unused_layers no)
-			(net 56 "unconnected-(U1-3V3_EN-Pad37)_1")
+			(net 54 "unconnected-(U1-3V3_EN-Pad37)_1")
 			(pinfunction "3V3_EN")
 			(pintype "input+no_connect")
@@
 			)
 			(layers "F.Cu" "F.Mask")
-			(net 55 "unconnected-(U1-3V3_EN-Pad37)")
+			(net 54 "unconnected-(U1-3V3_EN-Pad37)_1")
 			(pinfunction "3V3_EN")
 			(pintype "input+no_connect")
@@
 			(layers "*.Cu" "*.Mask")
 			(remove_unused_layers no)
-			(net 61 "unconnected-(U1-VBUS-Pad40)_1")
+			(net 57 "unconnected-(U1-VBUS-Pad40)_1")
 			(pinfunction "VBUS")
 			(pintype "bidirectional+no_connect")
@@
 			)
 			(layers "F.Cu" "F.Mask")
-			(net 54 "unconnected-(U1-VBUS-Pad40)")
+			(net 57 "unconnected-(U1-VBUS-Pad40)_1")
 			(pinfunction "VBUS")
 			(pintype "bidirectional+no_connect")
@@
 			(layers "*.Cu" "*.Mask")
 			(remove_unused_layers no)
-			(net 65 "unconnected-(U1-SWCLK-Pad41)")
+			(net 61 "unconnected-(U1-SWCLK-Pad41)")
 			(pinfunction "SWCLK")
 			(pintype "input+no_connect")
@@
 			(layers "*.Cu" "*.Mask")
 			(remove_unused_layers no)
-			(net 66 "unconnected-(U1-GND-Pad42)")
+			(net 62 "unconnected-(U1-GND-Pad42)")
 			(pinfunction "GND")
 			(pintype "power_in+no_connect")
@@
 			(layers "*.Cu" "*.Mask")
 			(remove_unused_layers no)
-			(net 64 "unconnected-(U1-SWDIO-Pad43)")
+			(net 60 "unconnected-(U1-SWDIO-Pad43)")
 			(pinfunction "SWDIO")
 			(pintype "bidirectional+no_connect")
@@
 			)
 		)
-		(model "${KIPRJMOD}/3d/RaspBerryPi_Pico_W.step"
+		(model "${KIPRJMOD}/Library.pretty/RaspBerryPi_Pico_W.step"
 			(offset
-				(xyz 0 25.5 0)
+				(xyz 0 25.5 -0.5)
 			)
 			(scale
@@
 			(size 3.5 3.5)
 			(drill 3.5)
-			(layers "F&B.Cu" "*.Mask")
+			(layers "*.Cu" "*.Mask")
 		)
 	)
@@
 			(layers "*.Cu" "*.Mask")
 			(remove_unused_layers no)
-			(net 68 "Net-(D10-K)")
+			(net 64 "Net-(D10-K)")
 			(pintype "passive")
 		)
@@
 			(layers "*.Cu" "*.Mask")
 			(remove_unused_layers no)
-			(net 63 "/DIGOUT1")
+			(net 59 "/DIGOUT1")
 			(pinfunction "1")
 			(pintype "passive")
@@
 			(layers "*.Cu" "*.Mask")
 			(remove_unused_layers no)
-			(net 67 "/LIGHT")
+			(net 63 "/LIGHT")
 			(pinfunction "5")
 			(pintype "passive")
@@
 			(pintype "passive")
 		)
-		(model "${KIPRJMOD}/3d/75915-416LF.step"
+		(model "${KIPRJMOD}/Library.pretty/75915-416LF.stp"
 			(offset
 				(xyz 0 0 0)
@@
 			(pintype "passive")
 		)
-		(model "${KIPRJMOD}/3d/RUEF090.step"
-			(offset
-				(xyz 2.5 0 4)
-			)
-			(scale
-				(xyz 1 1 1)
-			)
-			(rotate
-				(xyz -90 0 -20)
-			)
-		)
 		(model "${KIPRJMOD}/Library.pretty/RUEF090.step"
 			(offset
@@
 			)
 			(rotate
-				(xyz -90 0 -15)
+				(xyz -90 0 -20)
 			)
 		)
@@
 			(layers "*.Cu" "*.Mask")
 			(remove_unused_layers no)
-			(net 62 "unconnected-(J2-PadSHUNT)")
+			(net 58 "unconnected-(J2-PadSHUNT)")
 			(pintype "passive+no_connect")
 		)
@@
 			(pintype "passive")
 		)
-		(model "${KIPRJMOD}/3d/RAPC722X.step"
+		(model "${KIPRJMOD}/Library.pretty/RAPC722X.step"
 			(offset
 				(xyz 0 0 0)
@@
 			)
 			(rotate
-				(xyz -90 0 0)
+				(xyz 90 180 180)
 			)
 		)
@@
 			)
 		)
-		(fp_text user "K"
-			(at 0 -1.8 90)
+		(fp_text user "${REFERENCE}"
+			(at 4.11 0 90)
 			(layer "F.Fab")
 			(effects
 				(font
-					(size 1 1)
-					(thickness 0.15)
+					(size 0.8 0.8)
+					(thickness 0.12)
 				)
 			)
 		)
-		(fp_text user "${REFERENCE}"
-			(at 4.11 0 90)
+		(fp_text user "K"
+			(at 0 -1.8 90)
 			(layer "F.Fab")
 			(effects
 				(font
-					(size 0.8 0.8)
-					(thickness 0.12)
+					(size 1 1)
+					(thickness 0.15)
 				)
 			)
@@
 			(layers "*.Cu" "*.Mask")
 			(remove_unused_layers no)
-			(net 69 "Net-(U1-GPIO15)")
+			(net 65 "Net-(U1-GPIO15)")
 			(pinfunction "1")
 			(pintype "passive")
@@
 			(layers "*.Cu" "*.Mask")
 			(remove_unused_layers no)
-			(net 68 "Net-(D10-K)")
+			(net 64 "Net-(D10-K)")
 			(pinfunction "K")
 			(pintype "passive")
@@
 			(layers "*.Cu" "*.Mask")
 			(remove_unused_layers no)
-			(net 63 "/DIGOUT1")
+			(net 59 "/DIGOUT1")
 			(pinfunction "11")
 			(pintype "passive")
@@
 			(solder_mask_margin 0.102)
 		)
-		(model "${KIPRJMOD}/3d/10090926-P154XLF.step"
+		(model "${KIPRJMOD}/Library.pretty/10090926-P154XLF.step"
 			(offset
 				(xyz 0 0 0)
@@
 			)
 		)
-		(fp_text user "K"
-			(at 0 -1.8 90)
+		(fp_text user "${REFERENCE}"
+			(at 4.11 0 90)
 			(layer "F.Fab")
 			(effects
 				(font
-					(size 1 1)
-					(thickness 0.15)
+					(size 0.8 0.8)
+					(thickness 0.12)
 				)
 			)
 		)
-		(fp_text user "${REFERENCE}"
-			(at 4.11 0 90)
+		(fp_text user "K"
+			(at 0 -1.8 90)
 			(layer "F.Fab")
 			(effects
 				(font
-					(size 0.8 0.8)
-					(thickness 0.12)
+					(size 1 1)
+					(thickness 0.15)
 				)
 			)
@@
 			(size 3.5 3.5)
 			(drill 3.5)
-			(layers "F&B.Cu" "*.Mask")
+			(layers "*.Cu" "*.Mask")
 		)
 	)
@@
 			)
 		)
-		(fp_text user "${REFERENCE}"
-			(at 4.11 0 90)
+		(fp_text user "K"
+			(at 0 -1.8 90)
 			(layer "F.Fab")
 			(effects
 				(font
-					(size 0.8 0.8)
-					(thickness 0.12)
+					(size 1 1)
+					(thickness 0.15)
 				)
 			)
 		)
-		(fp_text user "K"
-			(at 0 -1.8 90)
+		(fp_text user "${REFERENCE}"
+			(at 4.11 0 90)
 			(layer "F.Fab")
 			(effects
 				(font
-					(size 1 1)
-					(thickness 0.15)
+					(size 0.8 0.8)
+					(thickness 0.12)
 				)
 			)
@@
 		)
 	)
-	(gr_text "V 0.0.5 2024-09-26"
+	(gr_text "V 0.0.6 2024-10-26"
 		(at 107.1372 79.7052 0)
 		(layer "F.SilkS")
@@
 		(width 0.508)
 		(layer "F.Cu")
-		(net 63)
+		(net 59)
 	)
 	(segment
@@
 		(width 0.508)
 		(layer "F.Cu")
-		(net 63)
+		(net 59)
 	)
 	(segment
@@
 		(width 0.508)
 		(layer "F.Cu")
-		(net 67)
+		(net 63)
 	)
 	(segment
@@
 		(width 0.508)
 		(layer "F.Cu")
-		(net 67)
+		(net 63)
 	)
 	(segment
@@
 		(width 0.508)
 		(layer "B.Cu")
-		(net 68)
+		(net 64)
 	)
 	(segment
@@
 		(width 0.508)
 		(layer "B.Cu")
-		(net 68)
+		(net 64)
 	)
 	(segment
@@
 		(width 0.508)
 		(layer "F.Cu")
-		(net 69)
+		(net 65)
 	)
 	(zone
